Commit message: Grab Object Tool 추가 1. pybullet 카메라로 이미지, Depth 데이터 획득 2. Yolo 추론으로 오브젝트의 중앙좌표 획득 3.  오브젝트의 중앙 좌표로 중앙 좌표 Depth 값을 획득 4. 카메라 설정 값을 통해 카메라 좌표계 기준 오브젝트 좌표로 변환 5. 월드 좌표계 기준 오브젝트 좌표로 변환 6. 이 좌표로 로봇팔을 움직여 좌표에 도달한 경우 그리퍼를 닫음.

File: robot/pybullet_sim/urdfs/dofbot.urdf (robot description, URDF)
Before this commit: robot dofbot, 9 links, 8 joints
Joints:
- joint joint-ee: origin xyz=0 0 0.09 -> xyz=0 0 0.11
